Commit message: comit t

File: description/lidar.xacro (robot description, xacro)
@@ -4,7 +4,7 @@
         <origin xyz="0.022 0.0 0.116141" rpy="0 0 0"/>
         <parent link="base_link"/>
-        <child link="laser_frame"/>
+        <child link="laser_link_1"/>
     </joint>
-    <link name="laser_frame">
+    <link name="laser_link_1">
         <inertial>
           <origin xyz="0.0 0.0 0.012500000000000039" rpy="0 0 0"/>
@@ -26,5 +26,5 @@
         </collision>
       </link>
-    <gazebo reference="laser_frame">
+    <gazebo reference="laser_link_1">
         <material>Gazebo/Red</material>
         <sensor name="laser" type="ray">
@@ -50,5 +50,5 @@
                 </ros>
                 <output_type>sensor_msgs/LaserScan</output_type>
-                <frame_name>laser_frame</frame_name>
+                <frame_name>laser_link_1</frame_name>
             </plugin>
         </sensor>

File: description/robot.urdf.xacro (robot description, xacro)
@@ -1,4 +1,4 @@
 <?xml version="1.0"?>
-<robot xmlns:xacro="http://www.ros.org/wiki/xacro"  name="ammrry">
+<robot xmlns:xacro="http://www.ros.org/wiki/xacro"  name="amiio">
     <xacro:arg name="use_ros2_control" default="true"/>
     <xacro:arg name="sim_mode" default="false"/>

File: description/ros2_control.xacro (robot description, xacro)
@@ -11,5 +11,5 @@
                 <param name="baud_rate">57600</param>
                 <param name="timeout_ms">1000</param>
-                <param name="enc_counts_per_rev">3436</param>
+                <param name="enc_counts_per_rev">1000</param>
             </hardware>
             <joint name="left_wheel_joint">
